File: pcb/badge.kicad_sch (KiCad schematic)
At the start: 54 parts, among them J1 USB_C_Receptacle_USB2.0_16P, J2 Conn_01x02, J3 Conn_01x03, Q1 Si1308EDL, SW1 SW_Push, U1 RP2040, U2 AP2112K-3.3, U3 W25Q32JVSSIQ, Y1 12MHz

Commit message: More footprints
Parts:
- C1, C10, C11, C12, C13, C17, C18, C19, C2, C20, C21, C22, C23, C25: footprint (none) -> MAJCT168BB7105KTEA01:MAJx16
- C14, C15: value C -> 1uF; footprint (none) -> MAJCT168BB7105KTEA01:MAJx16
- C16, C3, C4, C5, C6, C7, C8, C9: footprint (none) -> footprint:CAPC2012X94N
- C24, C26: footprint (none) -> GMK316AB7475KLHT:CAPC3216X180N
- D2: footprint (none) -> VLMC3100-GS08:LEDM3528X185N
- J1: footprint (none) -> Connector_USB:USB_C_Receptacle_Amphenol_12401610E4-2A
- J2: footprint (none) -> Connector_PinHeader_1.00mm:PinHeader_1x02_P1.00mm_Horizontal
- J3, L1: footprint (none) -> Connector_PinHeader_1.00mm:PinHeader_1x03_P1.00mm_Horizontal
- U1: footprint IC57_RP2040 -> RP2040:IC57_RP2040
Changed lines of the file:
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@@
 			)
 		)
-		(property "Footprint" ""
+		(property "Footprint" "footprint:CAPC2012X94N"
 			(at 187.6552 121.92 0)
 			(effects
@@
 			)
 		)
-		(property "Footprint" ""
+		(property "Footprint" "MAJCT168BB7105KTEA01:MAJx16"
 			(at 258.7752 148.59 0)
 			(effects
@@
 			)
 		)
-		(property "Footprint" ""
+		(property "Footprint" "footprint:CAPC2012X94N"
 			(at 82.55 117.1448 0)
 			(effects
@@
 			)
 		)
-		(property "Value" "C"
+		(property "Value" "1uF"
 			(at 148.59 40.6399 0)
 			(effects
@@
 			)
 		)
-		(property "Footprint" ""
+		(property "Footprint" "MAJCT168BB7105KTEA01:MAJx16"
 			(at 145.7452 43.18 0)
 			(effects
@@
 			)
 		)
-		(property "Footprint" ""
+		(property "Footprint" "Connector_USB:USB_C_Receptacle_Amphenol_12401610E4-2A"
 			(at 78.74 52.07 0)
 			(effects
@@
 			)
 		)
-		(property "Footprint" ""
+		(property "Footprint" "MAJCT168BB7105KTEA01:MAJx16"
 			(at 115.57 136.1948 0)
 			(effects
@@
 			)
 		)
-		(property "Footprint" ""
+		(property "Footprint" "MAJCT168BB7105KTEA01:MAJx16"
 			(at 261.3152 76.2 0)
 			(effects
@@
 			)
 		)
-		(property "Footprint" "IC57_RP2040"
+		(property "Footprint" "RP2040:IC57_RP2040"
 			(at 173.99 29.21 0)
 			(effects
@@
 			)
 		)
-		(property "Footprint" ""
+		(property "Footprint" "MAJCT168BB7105KTEA01:MAJx16"
 			(at 104.14 179.3748 0)
 			(effects
@@
 			)
 		)
-		(property "Footprint" ""
+		(property "Footprint" "MAJCT168BB7105KTEA01:MAJx16"
 			(at 79.7052 171.45 0)
 			(effects
@@
 			)
 		)
-		(property "Footprint" ""
+		(property "Footprint" "MAJCT168BB7105KTEA01:MAJx16"
 			(at 268.9352 105.41 0)
 			(effects
@@
 			)
 		)
-		(property "Footprint" ""
+		(property "Footprint" "MAJCT168BB7105KTEA01:MAJx16"
 			(at 252.4252 77.47 0)
 			(effects
@@
 			)
 		)
-		(property "Footprint" ""
+		(property "Footprint" "Connector_PinHeader_1.00mm:PinHeader_1x03_P1.00mm_Horizontal"
 			(at 106.68 106.68 0)
 			(effects
@@
 			)
 		)
-		(property "Footprint" ""
+		(property "Footprint" "MAJCT168BB7105KTEA01:MAJx16"
 			(at 107.95 171.7548 0)
 			(effects
@@
 			)
 		)
-		(property "Footprint" ""
+		(property "Footprint" "footprint:CAPC2012X94N"
 			(at 174.9552 121.92 0)
 			(effects
@@
 			)
 		)
-		(property "Footprint" ""
+		(property "Footprint" "MAJCT168BB7105KTEA01:MAJx16"
 			(at 257.5052 105.41 0)
 			(effects
@@
 			)
 		)
-		(property "Footprint" ""
+		(property "Footprint" "MAJCT168BB7105KTEA01:MAJx16"
 			(at 104.14 194.6148 0)
 			(effects
@@
 		(on_board yes)
 		(dnp no)
-		(fields_autoplaced yes)
 		(property "Reference" "C14"
 			(at 107.95 27.9399 0)
@@
 			)
 		)
-		(property "Value" "C"
+		(property "Value" "1uF"
 			(at 107.95 30.4799 0)
 			(effects
@@
 					(size 1.27 1.27)
 				)
-				(justify left)
 			)
 		)
-		(property "Footprint" ""
+		(property "Footprint" "MAJCT168BB7105KTEA01:MAJx16"
 			(at 105.1052 33.02 0)
 			(effects
@@
 			)
 		)
-		(property "Footprint" ""
+		(property "Footprint" "MAJCT168BB7105KTEA01:MAJx16"
 			(at 272.7452 148.59 0)
 			(effects
@@
 			)
 		)
-		(property "Footprint" ""
+		(property "Footprint" "GMK316AB7475KLHT:CAPC3216X180N"
 			(at 56.8452 156.21 0)
 			(effects
@@
 			)
 		)
-		(property "Footprint" ""
+		(property "Footprint" "MAJCT168BB7105KTEA01:MAJx16"
 			(at 104.14 164.1348 0)
 			(effects
@@
 			)
 		)
-		(property "Footprint" ""
+		(property "Footprint" "GMK316AB7475KLHT:CAPC3216X180N"
 			(at 44.1452 171.45 0)
 			(effects
@@
 			)
 		)
-		(property "Footprint" ""
+		(property "Footprint" "Connector_PinHeader_1.00mm:PinHeader_1x02_P1.00mm_Horizontal"
 			(at 106.68 92.71 0)
 			(effects
@@
 			)
 		)
-		(property "Footprint" ""
+		(property "Footprint" "footprint:CAPC2012X94N"
 			(at 238.4552 121.92 0)
 			(effects
@@
 			)
 		)
-		(property "Footprint" ""
+		(property "Footprint" "MAJCT168BB7105KTEA01:MAJx16"
 			(at 107.95 156.5148 0)
 			(effects
@@
 			)
 		)
-		(property "Footprint" ""
+		(property "Footprint" "footprint:CAPC2012X94N"
 			(at 225.7552 121.92 0)
 			(effects
@@
 			)
 		)
-		(property "Footprint" ""
+		(property "Footprint" "footprint:CAPC2012X94N"
 			(at 200.3552 121.92 0)
 			(effects
@@
 			)
 		)
-		(property "Footprint" ""
+		(property "Footprint" "MAJCT168BB7105KTEA01:MAJx16"
 			(at 107.95 186.9948 0)
 			(effects
@@
 			)
 		)
-		(property "Footprint" ""
+		(property "Footprint" "footprint:CAPC2012X94N"
 			(at 245.11 105.7148 0)
 			(effects
@@
 			)
 		)
-		(property "Footprint" ""
+		(property "Footprint" "footprint:CAPC2012X94N"
 			(at 213.0552 121.92 0)
 			(effects
@@
 			)
 		)
-		(property "Footprint" ""
+		(property "Footprint" "VLMC3100-GS08:LEDM3528X185N"
 			(at 46.99 39.37 0)
 			(effects
@@
 			)
 		)
-		(property "Footprint" ""
+		(property "Footprint" "Connector_PinHeader_1.00mm:PinHeader_1x03_P1.00mm_Horizontal"
 			(at 48.26 162.56 0)
 			(effects

Commit message: Began schematic
Parts:
- GDEY0213F1: footprint (none) -> Connector_FFC-FPC:Hirose_FH12-24S-0.5SH_1x24-1MP_P0.50mm_Horizontal
- R1, R7: footprint (none) -> Resistor_SMD:R_01005_0402Metric
- R10: footprint (none) -> Resistor_SMD:R_0805_2012Metric
- R11: footprint (none) -> Resistor_SMD:R_2010_5025Metric
- R12, R4, R5, R6: footprint (none) -> Resistor_SMD:R_1206_3216Metric
- R2, R3: footprint (none) -> Resistor_SMD:R_1210_3225Metric
- R8: value R -> 1k; footprint (none) -> Resistor_SMD:R_0201_0603Metric
- R9: footprint (none) -> Resistor_SMD:R_0201_0603Metric
- SW1: footprint (none) -> GMK316AB7475KLHT:CAPC3216X180N
- Y1: footprint (none) -> FC4SDCBMF12.0-T1:CRYSTAL_HC49SDLF_FXT
Changed lines of the file:
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@@
 			)
 		)
-		(property "Footprint" ""
+		(property "Footprint" "Resistor_SMD:R_0805_2012Metric"
 			(at 33.782 96.52 90)
 			(effects
@@
 			)
 		)
-		(property "Footprint" ""
+		(property "Footprint" "Resistor_SMD:R_1206_3216Metric"
 			(at 265.43 127.508 90)
 			(effects
@@
 			)
 		)
-		(property "Footprint" ""
+		(property "Footprint" "Resistor_SMD:R_1206_3216Metric"
 			(at 104.14 44.958 90)
 			(effects
@@
 			)
 		)
-		(property "Footprint" ""
+		(property "Footprint" "Resistor_SMD:R_2010_5025Metric"
 			(at 45.212 185.42 90)
 			(effects
@@
 			)
 		)
-		(property "Footprint" ""
+		(property "Footprint" "Resistor_SMD:R_1210_3225Metric"
 			(at 255.27 57.912 90)
 			(effects
@@
 			)
 		)
-		(property "Footprint" ""
+		(property "Footprint" "Resistor_SMD:R_1210_3225Metric"
 			(at 255.27 49.022 90)
 			(effects
@@
 			)
 		)
-		(property "Value" "R"
+		(property "Value" "1k"
 			(at 49.53 33.0199 0)
 			(effects
@@
 			)
 		)
-		(property "Footprint" ""
+		(property "Footprint" "Resistor_SMD:R_0201_0603Metric"
 			(at 45.212 31.75 90)
 			(effects
@@
 			)
 		)
-		(property "Footprint" ""
+		(property "Footprint" "Resistor_SMD:R_01005_0402Metric"
 			(at 156.972 87.63 90)
 			(effects
@@
 			)
 		)
-		(property "Footprint" ""
+		(property "Footprint" "Resistor_SMD:R_01005_0402Metric"
 			(at 116.84 43.688 90)
 			(effects
@@
 			)
 		)
-		(property "Footprint" ""
+		(property "Footprint" "Resistor_SMD:R_1206_3216Metric"
 			(at 55.372 185.42 90)
 			(effects
@@
 			)
 		)
-		(property "Footprint" ""
+		(property "Footprint" "FC4SDCBMF12.0-T1:CRYSTAL_HC49SDLF_FXT"
 			(at 265.43 135.89 0)
 			(effects
@@
 			)
 		)
-		(property "Footprint" ""
+		(property "Footprint" "Resistor_SMD:R_1206_3216Metric"
 			(at 97.79 50.038 90)
 			(effects
@@
 			)
 		)
-		(property "Footprint" ""
+		(property "Footprint" "Connector_FFC-FPC:Hirose_FH12-24S-0.5SH_1x24-1MP_P0.50mm_Horizontal"
 			(at 134.62 148.59 0)
 			(effects
@@
 			)
 		)
-		(property "Footprint" ""
+		(property "Footprint" "GMK316AB7475KLHT:CAPC3216X180N"
 			(at 44.45 59.69 0)
 			(effects
@@
 			)
 		)
-		(property "Footprint" ""
+		(property "Footprint" "Resistor_SMD:R_0201_0603Metric"
 			(at 30.48 103.378 90)
 			(effects
