File: pcb/badge.kicad_pcb (KiCad board)
At the start: 2 copper layers, 52 parts, among them J1 USB_C_Receptacle_USB2.0_16P, J2 Conn_01x02, J3 Conn_01x03, Q1 Si1308EDL, SW1 SW_Push, U1 RP2040, U2 AP2112K-3.3, Y1 12MHz

Commit message: Saving before autorouting
Parts:
- C1, C10, C11, C12, C13, C14, C15, C16, C17, C18, C19, C2, C20, C21, C22, C23, C24, C25, C26, C3, C4, C5, C6, C7, C8, C9, D2, D3, D4, D5, GDEY0213F1, Q1, R1, R10, R11, R12, R2, R3, R4, R5, R6, R7, R8, R9, SW1, U1, U2, Y1: moved to B.Cu
- moved R4 95.9 mm to (167.5, 141.5), turned to 180 degrees
- moved R12 84.6 mm to (188.2, 120.3), turned to -90 degrees
- moved R6 82.4 mm to (182.2, 120.3), turned to -90 degrees
- moved R5 81.5 mm to (176.7, 120.3), turned to -90 degrees
- moved R2 69.6 mm to (187.1, 126.3), turned to 180 degrees
- moved R3 69.6 mm to (187.1, 130.5), turned to 180 degrees
- moved C21 68.9 mm to (131.7, 124.6), turned to 180 degrees
- moved C23 68.9 mm to (131.7, 132.4), turned to 180 degrees
- moved C25 68.9 mm to (131.7, 136.3), turned to 180 degrees
- moved C22 68.9 mm to (131.7, 128.5), turned to 180 degrees
- moved R10 61.7 mm to (181.1, 132.3), turned to 180 degrees
- moved C17 60.2 mm to (136.9, 124.6), turned to 180 degrees
- moved C18 60.2 mm to (136.9, 128.5), turned to 180 degrees
- moved C19 60.2 mm to (136.9, 132.4), turned to 180 degrees
- moved C20 60.2 mm to (136.9, 136.3), turned to 180 degrees
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Routing:
- net GND: track 0.00 -> 35.6 mm
- net 3.3V: track 0.00 -> 6.90 mm
- net XOUT: track 0.00 -> 4.43 mm
- net XIN: track 0.00 -> 4.38 mm
- net USB_BOOT: track 0.00 -> 3.07 mm
Other:
- board outline added: 77 x 75 mm

Commit message: Finished routing
Parts:
- moved R7 12.7 mm to (172.0, 121.5)
Routing:
- net GND: track 35.6 -> 341.3 mm, vias 0 -> 4
- net 3.3V: track 6.90 -> 173.9 mm, vias 0 -> 4
- net Net-(J1-CC2): track 0.00 -> 103.0 mm, vias 0 -> 5
- net PREVGH: track 0.00 -> 99.3 mm, vias 0 -> 2
- net RESE: track 0.00 -> 90.5 mm, vias 0 -> 2
- net USB_N: track 0.00 -> 87.4 mm, vias 0 -> 3
- net USB_P: track 0.00 -> 82.5 mm, vias 0 -> 3
- net GDR: track 0.00 -> 77.9 mm, vias 0 -> 2
- net /PREVGL: track 0.00 -> 69.1 mm
- net XOUT: track 4.43 -> 70.3 mm
- net Net-(GDEY0213F1-VSN): track 0.00 -> 59.9 mm
- net Net-(J1-CC1): track 0.00 -> 58.6 mm, vias 0 -> 1
- net 1.1V: track 0.00 -> 55.0 mm, vias 0 -> 4
- net Net-(GDEY0213F1-VSP): track 0.00 -> 54.1 mm
- net Net-(GDEY0213F1-VDD): track 0.00 -> 49.2 mm
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Other:
- board size 77 x 75 mm -> 77 x 86.5 mm

Commit message: Added sketches
Parts:
- added G***: LOGO, LOGO, F.Cu at (140.5, 129.0)
- added G***: LOGO, LOGO, F.Cu at (169.5, 129.5)
